File: SolarsellMPPT/Arduino-mini-328-Sch.brd (EAGLE design)
At the start: 100 x 80 mm, 22 parts, among them IC1 LM358N

Commit message: chage some PCB
Connections:
- new net S$1: LOAD.1
- net N$13: no longer LOAD.1
Routing:
- net N$13: track 10.3 -> 8.75 mm
- added copper zone on layer 16, net S$2
- removed copper zone on layer 1, net N$9
